Commit message: urdf file updated

File: snake_descrip/urdf/TestModule.urdf (robot description, URDF)
Before this commit: robot TestModule, 1 links, 0 joints
Links:
- added link head, mass 0.00301708508515438; collision mesh filename=package://TestModule/meshes/head.STL; visual mesh filename=package://TestModule/meshes/head.STL
- added link link1, mass 0.065417433868186; collision mesh filename=package://TestModule/meshes/link1.STL; visual mesh filename=package://TestModule/meshes/link1.STL
- added link link2, mass 0.065417429839142; collision mesh filename=package://TestModule/meshes/link2.STL; visual mesh filename=package://TestModule/meshes/link2.STL
- added link link3, mass 0.065417436974768; collision mesh filename=package://TestModule/meshes/link3.STL; visual mesh filename=package://TestModule/meshes/link3.STL
- added link link4, mass 0.0654174306029862; collision mesh filename=package://TestModule/meshes/link4.STL; visual mesh filename=package://TestModule/meshes/link4.STL
- added link link5, mass 0.0654174406564615; collision mesh filename=package://TestModule/meshes/link5.STL; visual mesh filename=package://TestModule/meshes/link5.STL
- added link link6, mass 0.0158896889808625; collision mesh filename=package://TestModule/meshes/link6.STL; visual mesh filename=package://TestModule/meshes/link6.STL
- link base_link: mass 0.395521671326912 -> 0.0495277420594313
Joints:
- added joint J1: type continuous, parent base_link, child link1, origin xyz=0 0.04109 0.0236 rpy=0 0 0, axis 0 0 1
- added joint J2: type continuous, parent base_link, child link2, origin xyz=0.023978 0.1245 0.0021 rpy=0 0 0, axis 0 0 1
- added joint J3: type prismatic, parent base_link, child link3, origin xyz=0.083481 0.18807 0.026367 rpy=3.1409 0.013637 3.1416, axis 0 0 1, limit lower=0 upper=0 effort=0 velocity=0
- added joint J4: type prismatic, parent base_link, child link4, origin xyz=0.08293 0.27486 0.0049189 rpy=1.5576 0.059977 1.3541, axis 0.95993 0.28025 0, limit lower=0 upper=0 effort=0 velocity=0
- added joint J5: type prismatic, parent base_link, child link5, origin xyz=0.12089 0.34566 0.046738 rpy=-2.9144 -0.0087873 -0.0020312, axis 0.87595 0.46913 -0.11243, limit lower=0 upper=0 effort=0 velocity=0
- added joint J6: type fixed, parent base_link, child link6, origin xyz=0.07013 0.41905 0.041164 rpy=-1.4718 0.22816 -1.1572, axis 0 0 0
- added joint base: type fixed, parent base_link, child head, origin xyz=0 0 0 rpy=0 0 0, axis 0 0 0

Commit message: urdf updated

File: snake_descrip/urdf/TestModule.urdf (robot description, URDF)
Before this commit: robot TestModule, 8 links, 7 joints
Links:
- link link2: mass 0.065417429839142 -> 0.0654174298565387
- link link3: mass 0.065417436974768 -> 0.0654174369747681
- link link4: mass 0.0654174306029862 -> 0.0654174306201065
- link link5: mass 0.0654174406564615 -> 0.0654174406564616
- link link6: mass 0.0158896889808625 -> 0.0158896889808624
Joints:
- joint J2: origin xyz=0.023978 0.1245 0.0021 rpy=0 0 0 -> xyz=0.023978 0.083408 -0.0215 rpy=1.5708 0 1.0654; parent base_link -> link1
- joint J3: limit lower=0 upper=0 effort=0 velocity=0 -> (none); origin xyz=0.083481 0.18807 0.026367 rpy=3.1409 0.013637 3.1416 -> xyz=0.084432 0.024267 0.021289 rpy=-1.5469 1.0653 -3.1134; parent base_link -> link2; type prismatic -> continuous
- joint J4: axis 0.95993 0.28025 0 -> 0 0 1; limit lower=0 upper=0 effort=0 velocity=0 -> (none); origin xyz=0.08293 0.27486 0.0049189 rpy=1.5576 0.059977 1.3541 -> xyz=0.0008435 0.086772 0.0215 rpy=-1.5708 -0.063594 1.7866; parent base_link -> link3; type prismatic -> continuous
- joint J5: axis 0.87595 0.46913 -0.11243 -> 0 0 1; limit lower=0 upper=0 effort=0 velocity=0 -> (none); origin xyz=0.12089 0.34566 0.046738 rpy=-2.9144 -0.0087873 -0.0020312 -> xyz=0.074667 0.046086 0.022465 rpy=1.8196 -1.3569 0.040747; parent base_link -> link4; type prismatic -> continuous
- joint J6: axis 0 0 0 -> 0 0 1; origin xyz=0.07013 0.41905 0.041164 rpy=-1.4718 0.22816 -1.1572 -> xyz=-0.050961 -0.070249 0.0215 rpy=1.5708 -0.02304 1.1686; parent base_link -> link5; type fixed -> continuous
